File: hw/sch_pcb/RFIQINT01A.kicad_pcb (KiCad board)
At the start: 2 copper layers, 60.5 x 50.3 mm, 48 parts, among them J1 Umin ... Umax, J2 SATA7-67491-1030, J3 HEADER_1x08, J4 SATA7-67491-1030, J5 HEADER_1x08, J6 SATA7-67491-1030, M1 HOLE, M2 HOLE, M3 HOLE, M4 HOLE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

Commit message: Ulozeni v novem formatu KiCAD. A smazani starych dat.
Parts:
- C1: value C/U -> 10uF/16V
- C11, C12, C13, C14, C15, C16, C4, C5, C6, C7: value C -> 100nF
- C17: value C -> 10uF
- L1: value INDUCTOR -> BLM21PG331SN1D
Connections:
- U1 pad 1: (no net) -> unconnected-(U1-Pad1)
- U1 pad 4: (no net) -> unconnected-(U1-Pad4)
- U2 pad 1: (no net) -> unconnected-(U2-Pad1)
- U2 pad 4: (no net) -> unconnected-(U2-Pad4)
Other:
- net class Default removed
