File: hw/sch_pcb/RFIQINT01B.kicad_sch (KiCad schematic)
At the start: 48 parts, among them J1 Umin ... Umax, J2 SATA7-67491-1030, J3 HEADER_1x08, J4 SATA7-67491-1030, J5 HEADER_1x08, J6 SATA7-67491-1030, M1 HOLE, M2 HOLE, M3 HOLE, M4 HOLE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

Commit message: Edit. #3  #2
Parts:
- removed J1: Umin ... Umax, Mlab_Pin_Headers:Straight_2x03, symbol RFIQINT01A-rescue:HEADER_2x03_PARALLEL-RESCUE-RFIQINT01A
- added J1: HEADER_2x04_PARALLEL, Mlab_Pin_Headers:Straight_2x04, symbol MLAB_HEADER:HEADER_2x04_PARALLEL
- C1: footprint Capacitors_SMD:C_1210_HandSoldering -> Capacitor_SMD:C_0805_2012Metric; UST_ID (none) -> 5c70984812875079b91f8bbe
- C10, C11, C12, C13, C14, C15, C16, C2, C3, C4, C5, C6, C7, C8, C9: footprint Mlab_C:SMD-0603 -> Capacitor_SMD:C_0603_1608Metric; UST_ID (none) -> 5c70984812875079b91f8bf2
- C17: value 10uF -> 10uF/16V; footprint Mlab_C:C_0805 -> Capacitor_SMD:C_0805_2012Metric; UST_ID (none) -> 5c70984812875079b91f8bbe
- D1: footprint Diodes_SMD:D_SMA -> Diode_SMD:D_SMA; UST_ID (none) -> 5c70984512875079b91f88ac
- J2, J4, J6: footprint Connectors:SATA-7_THT_VERT_2 -> Mlab_CON:SATA-7_THT_VERT_2; UST_ID (none) -> 5c70984712875079b91f8a7b
- J3, J5: footprint maxrez:IDC381-8-110 -> Mlab_CON:IDC381-8-110; UST_ID (none) -> 5c70984712875079b91f8b89
- L1: UST_ID (none) -> 5c70984712875079b91f8b8a
- R1, R13, R14, R2: value 83 -> 82; footprint Mlab_R:SMD-0603 -> Resistor_SMD:R_0603_1608Metric; UST_ID (none) -> 5c70984512875079b91f8955
- R10, R12, R3, R5, R6, R7, R8, R9: value 127 -> 130; footprint Mlab_R:SMD-0603 -> Resistor_SMD:R_0603_1608Metric; UST_ID (none) -> 5cd08b17128750448e4542b1
- R11, R4: footprint Mlab_R:SMD-0603 -> Resistor_SMD:R_0603_1608Metric; UST_ID (none) -> 5c70984512875079b91f8956
- U1, U2: footprint Housings_SOIC:SOIC-8_3.9x4.9mm_Pitch1.27mm -> Package_SO:SOIC-8_3.9x4.9mm_P1.27mm; UST_ID (none) -> 5c70984712875079b91f8b81
- U3: footprint TO_SOT_Packages_SMD:SOT-223-3_TabPin2 -> Package_TO_SOT_SMD:SOT-223-3_TabPin2; UST_ID (none) -> 5c70984712875079b91f8af9
Connections:
- net ADC3_N: now also J5.4; no longer J5.5
- net ADC3_P: now also J5.3; no longer J5.6
- net ADC4_N: now also J5.6; no longer J5.3
- net ADC4_P: now also J5.5; no longer J5.4
- net CLK_OUT2_N: now also J5.8; no longer J5.1
- net CLK_OUT2_P: now also J5.7; no longer J5.2
- net GND: now also J5.2, J1.1, J1.2, J1.7, J1.8; no longer J5.7
- net VCC: now also J5.1, J1.3, J1.4, J1.5, J1.6; no longer J5.8
